File: hw/sensor_brick_model/sensor_brick_model.kicad_pcb (KiCad board)
At the start: 2 copper layers, 32 x 16 mm, 13 parts, among them J1 Conn_01x04_Male, J2 Conn_01x06_Male, U1 BMI160

Commit message: Version 1A done
Parts:
- added JP1: ADDR, Jumper:SolderJumper-3_P1.3mm_Bridged12_RoundedPad1.0x1.5mm, B.Cu at (126.4, 104.2)
- added R3: 10kR, Resistor_SMD:R_0603_1608Metric, F.Cu at (126.5, 106.2)
- C1, C2: value C_Small -> 100nF; footprint Capacitor_SMD:C_0402_1005Metric -> Capacitor_SMD:C_0603_1608Metric
- R1, R2: footprint Resistor_SMD:R_0402_1005Metric -> Resistor_SMD:R_0603_1608Metric
- TP1: value TestPoint -> 3V3
- TP2: value TestPoint -> SDA
- TP3: value TestPoint -> SCL
- TP4: value TestPoint -> GND
- moved C1 6.77 mm to (135.5, 106.8), turned to 0 degrees
- moved C2 0.79 mm to (135.0, 103.5), turned to 0 degrees
- moved R1 0.75 mm to (126.0, 100.0), turned to 270 degrees
- moved R2 0.75 mm to (138.0, 100.0), turned to 270 degrees
Connections:
- C1 pad 1: Net-(C1-Pad1) -> +3V3
- C1 pad 2: Net-(C1-Pad2) -> GND
- C2 pad 1: Net-(C2-Pad1) -> +3V3
- C2 pad 2: Net-(C2-Pad2) -> GND
- R1 pad 1: Net-(R1-Pad1) -> +3V3
- R2 pad 1: Net-(R1-Pad1) -> +3V3
- U1 pad 12: Net-(U1-Pad12) -> +3V3
- U1 pad 13: Net-(U1-Pad13) -> SCL
- U1 pad 14: Net-(U1-Pad14) -> SDA
- U1 pad 4: Net-(U1-Pad4) -> INT1
- U1 pad 5: Net-(U1-Pad5) -> +3V3
- U1 pad 6: Net-(U1-Pad6) -> GND
- U1 pad 7: Net-(U1-Pad7) -> GND
- U1 pad 8: Net-(U1-Pad8) -> +3V3
- U1 pad 9: Net-(U1-Pad9) -> INT2
Routing:
- net SCL: track 0.00 -> 22.3 mm
- net SDA: track 0.00 -> 21.2 mm
- net +3V3: track 0.00 -> 15.4 mm, vias 0 -> 4
- net INT2: track 0.00 -> 9.57 mm, vias 0 -> 1
- net INT1: track 0.00 -> 6.79 mm
- net Net-(JP1-Pad2): track 0.00 -> 5.54 mm, vias 0 -> 1
- net Net-(R3-Pad2): track 0.00 -> 4.17 mm
- net GND: track 0.00 -> 3.44 mm, vias 0 -> 3
- added copper zone on B.Cu, net +3V3
- added copper zone on F.Cu, net GND
Other:
- net class Default: clearance 0.2 -> 0.127; trace_width 0.25 -> 0.127; via_dia 0.8 -> 0.6; via_drill 0.4 -> 0.3
- net class USB added: clearance 0.3048, trace_width 0.1524, via_dia 0.6, via_drill 0.3
- net class USB_HS added: clearance 0.6096, trace_width 0.1524, via_dia 0.6, via_drill 0.3
- rule trace_clearance: 0.2 -> 0.127
- rule trace_min: 0.2 -> 0.127
- rule via_min_size: 0.4 -> 0.6
- board text added: "0x69 0x68"
- board text added: "3V3"
- board text added: "CodFish"
- board text added: "Designed in Portugal"
- board text added: "GND"
- board text added: "SCL"
- board text added: "SDA"
